Commit message: wip

File: dsr_description2/xacro/h2017.urdf.xacro (robot description, xacro)
@@ -18,7 +18,7 @@
   </xacro:if>
   <!-- World fixed joint-->
-  <joint name="world_fixed" type="fixed">
+  <joint name="base_base_0" type="fixed">
     <origin xyz="0 0 0" rpy="0 0 0"/>
-    <parent link="world"/>
+    <parent link="base"/>
     <child link="base_0"/>
   </joint>

File: dsr_description2/xacro/h2515.urdf.xacro (robot description, xacro)
@@ -21,5 +21,5 @@
     <origin xyz="0 0 0" rpy="0 0 0"/>
     <parent link="world"/>
-    <child link="base_0"/>
+    <child link="base"/>
   </joint>
 </robot>
