Commit message: Update Limits and urdf file

File: dsr_description2/xacro/macro.h2017.blue.xacro (robot description, xacro)
@@ -1,6 +1,4 @@
 <?xml version="1.0"?>
 <robot name="h2017" xmlns:xacro="http://www.ros.org/wiki/xacro">
-	<xacro:include filename="$(find dsr_description2)/config/macro.gazebo.xacro" />
-	<xacro:include filename="$(find dsr_description2)/config/macro.transmission.xacro" />
 	<!--xacro:include filename="$(find dsr_description2)/config/macro.materials.xacro" /-->
 	<xacro:macro name="h2017" params="namespace">
@@ -203,6 +201,4 @@
 			</visual>
 		</link>
-		<xacro:dsr_transmission />
-		<xacro:dsr_gazebo namespace="${namespace}" />
 	</xacro:macro>
 </robot>

File: moveit_config_h2017/config/h2017.urdf.xacro (robot description, xacro)
@@ -4,5 +4,12 @@
     <xacro:arg name="name" default="h2017" />
     <!-- Import h2017 urdf file -->
-    <xacro:include filename="$(find dsr_description2)/urdf/h2017.blue.urdf" />
+    <xacro:include filename="$(find dsr_description2)/xacro/macro.h2017.blue.xacro" />
+    <xacro:h2017 namespace=""/>
+    <!-- World fixed joint-->
+    <joint name="base_base_0" type="fixed">
+      <origin xyz="0 0 0" rpy="0 0 0"/>
+      <parent link="base"/>
+      <child link="base_0"/>
+    </joint>
     <!-- Import control_xacro -->
     <xacro:include filename="h2017.ros2_control.xacro" />

Commit message: Updates to doosan

File: dsr_description2/xacro/macro.h2017.blue.xacro (robot description, xacro)
@@ -18,4 +18,9 @@
 				</geometry>
 			</visual>
+      <collision>
+          <geometry>
+              <cylinder radius="0.0" length="0.0"/>
+          </geometry>
+      </collision>
 		</link>
 		<!-- joint 1 -->
@@ -111,4 +116,9 @@
 				</geometry>
 			</visual>
+      <collision>
+          <geometry>
+              <cylinder radius="0.0" length="0.0"/>
+          </geometry>
+      </collision>
 		</link>
 		<!-- joint4 -->
@@ -200,4 +210,10 @@
 				</geometry>
 			</visual>
+      <collision>
+          <origin rpy="0 0 0" xyz="0 0 0" />
+          <geometry>
+              <cylinder radius="0.00" length="0.0"/>
+          </geometry>
+      </collision>
 		</link>
 	</xacro:macro>
