Commit message: update h2017

File: dsr_description2/urdf/h2017.white.urdf (robot description, URDF)
Before this commit: robot h2017, 8 links, 7 joints
Links:
- link base_0: geometry collision mesh filename=package://dsr_description2/meshes/h2017_white/H2017_0_0.dae scale=0.001 0.001 0.001; visual mesh filename=package://dsr_description2/meshes/h2017_white/H2017_0_0.dae scale=0.001 0.001 0.001
- link link1: geometry collision mesh filename=package://dsr_description2/meshes/h2017_white/H2017_1_0.dae scale=0.001 0.001 0.001; visual mesh filename=package://dsr_description2/meshes/h2017_white/H2017_1_0.dae scale=0.001 0.001 0.001
- link link2: geometry collision mesh filename=package://dsr_description2/meshes/h2017_white/H2017_2_0.dae scale=0.001 0.001 0.001; collision mesh filename=package://dsr_description2/meshes/h2017_white/H2017_2_1.dae scale=0.001 0.001 0.001
- link link3: geometry collision mesh filename=package://dsr_description2/meshes/h2017_white/H2017_3_0.dae scale=0.001 0.001 0.001; visual mesh filename=package://dsr_description2/meshes/h2017_white/H2017_3_0.dae scale=0.001 0.001 0.001
- link link4: geometry collision mesh filename=package://dsr_description2/meshes/h2017_white/H2017_4_0.dae scale=0.001 0.001 0.001; collision mesh filename=package://dsr_description2/meshes/h2017_white/H2017_4_1.dae scale=0.001 0.001 0.001
- link link5: geometry collision mesh filename=package://dsr_description2/meshes/h2017_white/H2017_5_0.dae scale=0.001 0.001 0.001; visual mesh filename=package://dsr_description2/meshes/h2017_white/H2017_5_0.dae scale=0.001 0.001 0.001
- link link6: geometry collision mesh filename=package://dsr_description2/meshes/h2017_white/H2017_6_0.dae scale=0.001 0.001 0.001; visual mesh filename=package://dsr_description2/meshes/h2017_white/H2017_6_0.dae scale=0.001 0.001 0.001
